File: PCB/PCB.kicad_pcb (KiCad board)
At the start: 2 copper layers, 14 parts, among them J1 Conn_01x08_Pin, J2 Conn_01x02_Socket, K1 SANYOU_SRD_Form_B, Q1 NPN, SW1 SW_Push, U2 L7805

Commit message: PCB design done
Parts:
- added J3: Lock 12V output, Connector_PinSocket_2.54mm:PinSocket_1x02_P2.54mm_Vertical, F.Cu at (220.5, 100.5)
- added U1: XIAO-ESP32-C3-SMD, Imported Parts:XIAO-ESP32-C3-SMD, F.Cu at (145.2, 79.0)
- BZ1: footprint Buzzer_Beeper:Buzzer_15x7.5RM7.6 -> Buzzer_Beeper:Buzzer_12x9.5RM7.6
- D1: footprint LED_THT:LED_D1.8mm_W1.8mm_H2.4mm_Horizontal_O1.27mm_Z4.9mm -> LED_THT:LED_D1.8mm_W3.3mm_H2.4mm
- D2: footprint LED_THT:LED_D1.8mm_W1.8mm_H2.4mm_Horizontal_O3.81mm_Z4.9mm -> LED_THT:LED_D1.8mm_W3.3mm_H2.4mm
- J1: value Conn_01x08_Pin -> RFID connector
- J2: value Conn_01x02_Socket -> 12V alim connexion
- Q1: footprint Transistor_Power:GaN_Systems_GaNPX-3_5x6.6mm_Drain3.76x0.6mm -> Connector_PinHeader_2.54mm:PinHeader_1x03_P2.54mm_Vertical
- SW1: footprint Button_Switch_THT:SW_PUSH_6mm_H5mm -> Connector_PinHeader_2.54mm:PinHeader_1x02_P2.54mm_Vertical
- U2: footprint Transistor_Power:GaN_Systems_GaNPX-3_5x6.6mm_Drain2.93x0.6mm -> Connector_PinHeader_2.54mm:PinHeader_1x03_P2.54mm_Vertical
- moved Q1 102.9 mm to (193.0, 83.3), turned to 180 degrees
- moved K1 96.5 mm to (189.0, 103.7)
- moved C1 89.7 mm to (177.1, 55.6), turned to -90 degrees
- moved U2 81.1 mm to (169.1, 48.1), turned to -90 degrees
- moved R2 71.7 mm to (171.2, 80.7)
- moved BZ1 69.5 mm to (85.2, 79.0), turned to 90 degrees
- moved J2 68.2 mm to (188.1, 55.8)
- moved C2 65.2 mm to (157.1, 55.9), turned to -90 degrees
- moved D1 58.3 mm to (108.9, 76.0), turned to -90 degrees
- moved SW1 44.5 mm to (158.2, 71.0), turned to 180 degrees
- moved J1 37.3 mm to (77.2, 94.6)
- moved D3 31.1 mm to (168.0, 110.8), turned to 90 degrees
- moved D2 24.1 mm to (100.9, 76.0), turned to -90 degrees
- moved R1 15.3 mm to (104.4, 68.5), turned to 90 degrees
Connections:
- BZ1 pad 1: /GPIO3 -> /GPIO4
- D2 pad 2: /GPIO4 -> /GPIO3
Routing:
- net GND: track 0.00 -> 243.8 mm
- net +3.3V: track 0.00 -> 157.7 mm
- net +5V: track 0.00 -> 126.7 mm
- net +12V: track 0.00 -> 102.4 mm
- net /SCL: track 0.00 -> 72.6 mm
- net /SDA: track 0.00 -> 66.9 mm
- net Net-(D3-A): track 0.00 -> 54.0 mm
- net /GPIO4: track 0.00 -> 48.3 mm
- net /GPIO21: track 0.00 -> 30.0 mm
- net /GPIO3: track 0.00 -> 29.9 mm
- net /GPIO5: track 0.00 -> 26.4 mm
- net Net-(D1-K): track 0.00 -> 18.4 mm
- net /GPIO2: track 0.00 -> 18.3 mm
- net Net-(Q1-B): track 0.00 -> 14.2 mm
Other:
- board outline added: 155.5 x 75.5 mm

Commit message: Pcb remaked to use SPI instead of I2C
Connections:
- J1 pad 1: /SDA -> unconnected-(J1-Pin_1-Pad1)
- J1 pad 2: unconnected-(J1-Pin_2-Pad2) -> /SCK
- J1 pad 3: unconnected-(J1-Pin_3-Pad3) -> /MOSI
- J1 pad 4: /SCL -> /MISO
- U1 pad 10: unconnected-(U1-D9/BOOT-Pad10) -> /MISO
- U1 pad 11: unconnected-(U1-D10-Pad11) -> /MOSI
- U1 pad 5: /SDA -> unconnected-(U1-D4-Pad5)
- U1 pad 6: /SCL -> unconnected-(U1-D5-Pad6)
- U1 pad 9: unconnected-(U1-D8-Pad9) -> /SCK
Routing:
- net +5V: track 126.7 -> 303.9 mm
- net /MISO: track 0.00 -> 101.9 mm
- net /SCK: track 0.00 -> 91.7 mm
- net /MOSI: track 0.00 -> 86.1 mm
- net GND: track 243.8 -> 327.5 mm
- net /SCL: track 72.6 -> 0.00 mm
- net /SDA: track 66.9 -> 0.00 mm
- net +3.3V: track 157.7 -> 93.6 mm
