File: PCB/PCB.kicad_sch (KiCad schematic)
At the start: 15 parts, among them J1 Conn_01x08_Pin, J2 Conn_01x02_Socket, K1 SANYOU_SRD_Form_B, Q1 NPN, SW1 SW_Push, U1 XIAO-ESP32-C3-SMD, U2 L7805

Commit message: PCB design done
Parts:
- added J3: Lock 12V output, Connector_PinSocket_2.54mm:PinSocket_1x02_P2.54mm_Vertical, symbol Connector:Conn_01x02_Socket
- BZ1: footprint Buzzer_Beeper:Buzzer_15x7.5RM7.6 -> Buzzer_Beeper:Buzzer_12x9.5RM7.6
- D1: footprint LED_THT:LED_D1.8mm_W1.8mm_H2.4mm_Horizontal_O1.27mm_Z4.9mm -> LED_THT:LED_D1.8mm_W3.3mm_H2.4mm
- D2: footprint LED_THT:LED_D1.8mm_W1.8mm_H2.4mm_Horizontal_O3.81mm_Z4.9mm -> LED_THT:LED_D1.8mm_W3.3mm_H2.4mm
- J1: value Conn_01x08_Pin -> RFID connector
- J2: value Conn_01x02_Socket -> 12V alim connexion
- Q1: footprint Transistor_Power:GaN_Systems_GaNPX-3_5x6.6mm_Drain3.76x0.6mm -> Connector_PinHeader_2.54mm:PinHeader_1x03_P2.54mm_Vertical
- SW1: footprint Button_Switch_THT:SW_PUSH_6mm_H5mm -> Connector_PinHeader_2.54mm:PinHeader_1x02_P2.54mm_Vertical
- U1: footprint Seeed_Studio_XIAO_Series:XIAO-ESP32-C3-SMD -> Imported Parts:XIAO-ESP32-C3-SMD
- U2: footprint Transistor_Power:GaN_Systems_GaNPX-3_5x6.6mm_Drain2.93x0.6mm -> Connector_PinHeader_2.54mm:PinHeader_1x03_P2.54mm_Vertical
Connections:
- net +12V: now also J3.2 (Pin_2)
- net GND: now also J3.1 (Pin_1)
- net GPIO3: now also D2.2 (A); no longer BZ1.1 (+)
- net GPIO4: now also BZ1.1 (+); no longer D2.2 (A)
Changed lines of the file:
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@@
 	)
 	(junction
+		(at 209.55 76.2)
+		(diameter 0)
+		(color 0 0 0 0)
+	)
+	(junction
 		(at 199.39 85.09)
 		(diameter 0)
 		(color 0 0 0 0)
 	)
+	(junction
+		(at 209.55 60.96)
+		(diameter 0)
+		(color 0 0 0 0)
+	)
 	(no_connect
 		(at 148.59 63.5)
@@
 	(wire
 		(pts
+			(xy 243.84 68.58) (xy 243.84 60.96)
+		)
+		(stroke
+			(width 0)
+			(type default)
+		)
+	)
+	(wire
+		(pts
 			(xy 92.71 119.38) (xy 102.87 119.38)
 		)
@@
 	(wire
 		(pts
+			(xy 243.84 60.96) (xy 209.55 60.96)
+		)
+		(stroke
+			(width 0)
+			(type default)
+		)
+	)
+	(wire
+		(pts
 			(xy 118.11 119.38) (xy 118.11 125.73)
 		)
@@
 	(wire
 		(pts
+			(xy 243.84 76.2) (xy 209.55 76.2)
+		)
+		(stroke
+			(width 0)
+			(type default)
+		)
+	)
+	(wire
+		(pts
 			(xy 148.59 58.42) (xy 158.75 58.42)
 		)
@@
 	(wire
 		(pts
+			(xy 243.84 71.12) (xy 243.84 76.2)
+		)
+		(stroke
+			(width 0)
+			(type default)
+		)
+	)
+	(wire
+		(pts
 			(xy 137.16 101.6) (xy 144.78 101.6)
 		)
@@
 		)
 	)
-	(label "GPIO3"
+	(label "GPIO4"
 		(at 137.16 96.52 0)
 		(effects
@@
 		)
 	)
-	(label "GPIO4"
+	(label "GPIO3"
 		(at 92.71 130.81 0)
 		(effects
@@
 	)
 	(symbol
+		(lib_id "Connector:Conn_01x02_Socket")
+		(at 248.92 68.58 0)
+		(unit 1)
+		(body_style 1)
+		(exclude_from_sim no)
+		(in_bom yes)
+		(on_board yes)
+		(in_pos_files yes)
+		(dnp no)
+		(fields_autoplaced yes)
+		(property "Reference" "J3"
+			(at 250.19 68.5799 0)
+			(show_name no)
+			(do_not_autoplace no)
+			(effects
+				(font
+					(size 1.27 1.27)
+				)
+				(justify left)
+			)
+		)
+		(property "Value" "Lock 12V output"
+			(at 250.19 71.1199 0)
+			(show_name no)
+			(do_not_autoplace no)
+			(effects
+				(font
+					(size 1.27 1.27)
+				)
+				(justify left)
+			)
+		)
+		(property "Footprint" "Connector_PinSocket_2.54mm:PinSocket_1x02_P2.54mm_Vertical"
+			(at 248.92 68.58 0)
+			(hide yes)
+			(show_name no)
+			(do_not_autoplace no)
+			(effects
+				(font
+					(size 1.27 1.27)
+				)
+			)
+		)
+		(property "Datasheet" ""
+			(at 248.92 68.58 0)
+			(hide yes)
+			(show_name no)
+			(do_not_autoplace no)
+			(effects
+				(font
+					(size 1.27 1.27)
+				)
+			)
+		)
+		(property "Description" "Generic connector, single row, 01x02, script generated"
+			(at 248.92 68.58 0)
+			(hide yes)
+			(show_name no)
+			(do_not_autoplace no)
+			(effects
+				(font
+					(size 1.27 1.27)
+				)
+			)
+		)
+		(pin "1"
+		)
+		(pin "2"
+		)
+		(instances
+			(project "PCB"
+				(path "/e1ff644c-7932-4f1d-b11d-2ceea14cdfcd"
+					(reference "J3")
+					(unit 1)
+				)
+			)
+		)
+	)
+	(symbol
 		(lib_id "Seeed_Studio_XIAO_Series:XIAO-ESP32-C3-SMD")
 		(at 83.82 68.58 0)
@@
 			)
 		)
-		(property "Footprint" "Seeed_Studio_XIAO_Series:XIAO-ESP32-C3-SMD"
+		(property "Footprint" "Imported Parts:XIAO-ESP32-C3-SMD"
 			(at 45.212 92.964 0)
 			(hide yes)
@@
 			)
 		)
-		(property "Footprint" "Buzzer_Beeper:Buzzer_15x7.5RM7.6"
+		(property "Footprint" "Buzzer_Beeper:Buzzer_12x9.5RM7.6"
 			(at 146.685 96.52 90)
 			(hide yes)
@@
 			)
 		)
-		(property "Footprint" "LED_THT:LED_D1.8mm_W1.8mm_H2.4mm_Horizontal_O3.81mm_Z4.9mm"
+		(property "Footprint" "LED_THT:LED_D1.8mm_W3.3mm_H2.4mm"
 			(at 106.68 130.81 0)
 			(hide yes)
@@
 			)
 		)
-		(property "Footprint" "LED_THT:LED_D1.8mm_W1.8mm_H2.4mm_Horizontal_O1.27mm_Z4.9mm"
+		(property "Footprint" "LED_THT:LED_D1.8mm_W3.3mm_H2.4mm"
 			(at 106.68 119.38 0)
 			(hide yes)
@@
 			)
 		)
-		(property "Value" "Conn_01x08_Pin"
+		(property "Value" "RFID connector"
 			(at 144.145 55.88 0)
 			(show_name no)
@@
 			)
 		)
-		(property "Value" "Conn_01x02_Socket"
+		(property "Value" "12V alim connexion"
 			(at 149.86 149.8599 0)
 			(show_name no)
@@
 			)
 		)
-		(property "Footprint" "Transistor_Power:GaN_Systems_GaNPX-3_5x6.6mm_Drain2.93x0.6mm"
+		(property "Footprint" "Connector_PinHeader_2.54mm:PinHeader_1x03_P2.54mm_Vertical"
 			(at 231.775 118.11 0)
 			(hide yes)
@@
 			)
 		)
-		(property "Footprint" "Button_Switch_THT:SW_PUSH_6mm_H5mm"
+		(property "Footprint" "Connector_PinHeader_2.54mm:PinHeader_1x02_P2.54mm_Vertical"
 			(at 175.26 119.38 0)
 			(hide yes)
@@
 			)
 		)
-		(property "Footprint" "Transistor_Power:GaN_Systems_GaNPX-3_5x6.6mm_Drain3.76x0.6mm"
+		(property "Footprint" "Connector_PinHeader_2.54mm:PinHeader_1x03_P2.54mm_Vertical"
 			(at 233.68 29.21 0)
 			(hide yes)

Commit message: Pcb remaked to use SPI instead of I2C
Connections:
- net MISO: now reaches U1.10 (D9/BOOT)
- net MISO: now also J1.4 (Pin_4)
- net MOSI: now reaches U1.11 (D10)
- net MOSI: now also J1.3 (Pin_3)
- net SCK: now reaches U1.9 (D8)
- net SCK: now also J1.2 (Pin_2)
- net SCL: no longer names the net of U1.6 (D5)
- net SCL: no longer J1.4 (Pin_4)
- net SDA: no longer names the net of U1.5 (D4)
- net SDA: no longer J1.1 (Pin_1)
- no-connect marks 4 -> 0
Changed lines of the file:
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@@
 		(color 0 0 0 0)
 	)
-	(no_connect
-		(at 148.59 63.5)
-	)
-	(no_connect
-		(at 148.59 68.58)
-	)
-	(no_connect
-		(at 148.59 60.96)
-	)
-	(no_connect
-		(at 148.59 73.66)
-	)
 	(wire
 		(pts
@@
 	(wire
 		(pts
+			(xy 104.14 80.01) (xy 111.76 80.01)
+		)
+		(stroke
+			(width 0)
+			(type default)
+		)
+	)
+	(wire
+		(pts
 			(xy 209.55 76.2) (xy 209.55 82.55)
 		)
@@
 	(wire
 		(pts
+			(xy 148.59 66.04) (xy 156.21 66.04)
+		)
+		(stroke
+			(width 0)
+			(type default)
+		)
+	)
+	(wire
+		(pts
 			(xy 180.34 124.46) (xy 186.69 124.46)
 		)
@@
 	(wire
 		(pts
+			(xy 104.14 76.2) (xy 111.76 76.2)
+		)
+		(stroke
+			(width 0)
+			(type default)
+		)
+	)
+	(wire
+		(pts
 			(xy 133.35 147.32) (xy 143.51 147.32)
 		)
@@
 	(wire
 		(pts
+			(xy 104.14 72.39) (xy 111.76 72.39)
+		)
+		(stroke
+			(width 0)
+			(type default)
+		)
+	)
+	(wire
+		(pts
 			(xy 125.73 125.73) (xy 130.81 125.73)
 		)
@@
 	(wire
 		(pts
-			(xy 53.34 76.2) (xy 62.23 76.2)
-		)
-		(stroke
-			(width 0)
-			(type default)
-		)
-	)
-	(wire
-		(pts
 			(xy 215.9 114.3) (xy 223.52 114.3)
 		)
@@
 	(wire
 		(pts
-			(xy 148.59 66.04) (xy 158.75 66.04)
-		)
-		(stroke
-			(width 0)
-			(type default)
-		)
-	)
-	(wire
-		(pts
-			(xy 53.34 80.01) (xy 62.23 80.01)
+			(xy 148.59 63.5) (xy 156.21 63.5)
+		)
+		(stroke
+			(width 0)
+			(type default)
+		)
+	)
+	(wire
+		(pts
+			(xy 148.59 60.96) (xy 156.21 60.96)
 		)
 		(stroke
@@
 		(pts
 			(xy 243.84 76.2) (xy 209.55 76.2)
-		)
-		(stroke
-			(width 0)
-			(type default)
-		)
-	)
-	(wire
-		(pts
-			(xy 148.59 58.42) (xy 158.75 58.42)
 		)
 		(stroke
@@
 		)
 	)
+	(label "MISO"
+		(at 156.21 66.04 0)
+		(effects
+			(font
+				(size 1.27 1.27)
+			)
+			(justify left bottom)
+		)
+	)
 	(label "GPIO21"
 		(at 55.88 83.82 0)
@@
 		)
 	)
+	(label "MOSI"
+		(at 156.21 63.5 0)
+		(effects
+			(font
+				(size 1.27 1.27)
+			)
+			(justify left bottom)
+		)
+	)
 	(label "GPIO5"
 		(at 161.29 124.46 0)
@@
 		)
 	)
-	(label "SDA"
-		(at 158.75 58.42 0)
+	(label "MISO"
+		(at 111.76 76.2 0)
 		(effects
 			(font
@@
 		)
 	)
+	(label "SCK"
+		(at 156.21 60.96 0)
+		(effects
+			(font
+				(size 1.27 1.27)
+			)
+			(justify left bottom)
+		)
+	)
 	(label "GPIO2"
 		(at 92.71 119.38 0)
@@
 		)
 	)
+	(label "MOSI"
+		(at 111.76 72.39 0)
+		(effects
+			(font
+				(size 1.27 1.27)
+			)
+			(justify left bottom)
+		)
+	)
 	(label "GPIO5"
 		(at 54.61 72.39 0)
@@
 		)
 	)
-	(label "SCL"
-		(at 158.75 66.04 0)
-		(effects
-			(font
-				(size 1.27 1.27)
-			)
-			(justify left bottom)
-		)
-	)
-	(label "SDA"
-		(at 53.34 76.2 0)
-		(effects
-			(font
-				(size 1.27 1.27)
-			)
-			(justify left bottom)
-		)
-	)
-	(label "SCL"
-		(at 53.34 80.01 0)
+	(label "SCK"
+		(at 111.76 80.01 0)
 		(effects
 			(font
@@
 	(symbol
 		(lib_id "power:+3.3V")
-		(at 111.76 68.58 180)
+		(at 111.76 68.58 270)
 		(unit 1)
 		(body_style 1)
@@
 		(fields_autoplaced yes)
 		(property "Reference" "#PWR01"
-			(at 111.76 64.77 0)
+			(at 107.95 68.58 0)
 			(hide yes)
 			(show_name no)
@@
 		)
 		(property "Value" "+3.3V"
-			(at 111.76 73.66 0)
-			(show_name no)
-			(do_not_autoplace no)
-			(effects
-				(font
-					(size 1.27 1.27)
-				)
-			)
-		)
+			(at 115.57 68.5799 90)
+			(show_name no)
+			(do_not_autoplace no)
+			(effects
+				(font
+					(size 1.27 1.27)
+				)
+				(justify left)
+			)
+		)
